Commit message: added property unit comments. added pcb density property.

File: robot/millihex_description.xacro (robot description, xacro)
@@ -2,21 +2,23 @@
 <robot name="millihex" xmlns:xacro="http://www.ros.org/wiki/xacro">
     <!-- Physical Properties -->
-    <!-- Torso mass and x,y dimensions -->
+    <!-- PCB density ~ FR4 density (kg/m^3) -->
+    <xacro:property name="pcb_density" value="1850" />
+    <!-- Torso mass (kg) and x,y dimensions (m) -->
     <xacro:property name="torso_mass" value="0.01" />
     <xacro:property name="torso_x" value="0.14" />
     <xacro:property name="torso_y" value="0.04" />
-    <!-- Leg mass and x,y dimensions -->
+    <!-- Leg mass (kg) and x,y dimensions (m) -->
     <xacro:property name="leg_link_mass" value="0.0008" />
     <xacro:property name="leg_link_x" value="0.02" />
     <xacro:property name="leg_link_y" value="0.03" />
-    <!-- Joint limits -->
+    <!-- Joint limits (rad) -->
     <xacro:property name="joint_upper_limit" value="1.5708" />
     <xacro:property name="joint_lower_limit" value="-1.5708" />
     <xacro:property name="joint_effort_limit" value="0.01" />
     <xacro:property name="joint_velocity_limit" value="0.01" />
-    <!-- Joint damping (b) and friction (k) -->
+    <!-- Joint damping (b = N*s/m) and spring constant (k = N/m) -->
     <xacro:property name="joint_damping" value="0.00003" />
     <xacro:property name="joint_friction" value="0.001" />
-    <!-- PCB thickness -->
+    <!-- PCB thickness (m) -->
     <xacro:property name="pcb_thickness_z" value="0.0005" />
     <!-- Link Gazebo properties -->

Commit message: added equation macro to calculate mass of box. added command to convert xacro to urdf for testing equations

File: robot/millihex_description.xacro (robot description, xacro)
@@ -1,4 +1,16 @@
+<!-- Check URDF: -->
+<!-- rosrun xacro xacro millihex_description.xacro > millihex_description.urdf -->
 <?xml version="1.0"?>
 <robot name="millihex" xmlns:xacro="http://www.ros.org/wiki/xacro">
+    <!-- Equations -->
+    <!-- Calculate Mass of a Box -->
+    <xacro:macro name="box_mass" params="density x y z">
+        <mass value="${density*x*y*z}" />
+    </xacro:macro>
+    <!-- Calculate Moment of Inertia of a Box -->
+    <xacro:macro name="box_inertia" params="mass x y z">
+        <inertia ixx="${mass*(y*y+z*z)/12}" ixy = "0" ixz = "0"
+            iyy="${mass*(x*x+z*z)/12}" iyz = "0" izz="${mass*(x*x+y*y)/12}" />
+    </xacro:macro>
     <!-- Physical Properties -->
     <!-- PCB density ~ FR4 density (kg/m^3) -->
@@ -38,9 +50,4 @@
         <color rgba="0.98 0.41 0.055 1" />
     </material>
-    <!-- Calculate Moment of Inertia of a Box -->
-    <xacro:macro name="box_inertia" params="mass x y z">
-        <inertia ixx="${mass*(y*y+z*z)/12}" ixy = "0" ixz = "0"
-            iyy="${mass*(x*x+z*z)/12}" iyz = "0" izz="${mass*(x*x+y*y)/12}" />
-    </xacro:macro>
     <!-- Base and Torso Definition -->
     <xacro:macro name="millihex_torso" params="color">
@@ -248,5 +255,5 @@
         </gazebo>
     </xacro:macro>
-    <!-- Build Robot by Filling in Macro Parameters -->
+    <!-- Build Robot and Gazebo Control Library -->
     <xacro:millihex_body />
     <xacro:millihex_control namespace="millihex" />

Commit message: defined torso_mass and leg_link_mass properties

File: robot/millihex_description.xacro (robot description, xacro)
@@ -1,27 +1,21 @@
+<?xml version="1.0"?>
 <!-- Check URDF: -->
 <!-- rosrun xacro xacro millihex_description.xacro > millihex_description.urdf -->
-<?xml version="1.0"?>
 <robot name="millihex" xmlns:xacro="http://www.ros.org/wiki/xacro">
-    <!-- Equations -->
-    <!-- Calculate Mass of a Box -->
-    <xacro:macro name="box_mass" params="density x y z">
-        <mass value="${density*x*y*z}" />
-    </xacro:macro>
-    <!-- Calculate Moment of Inertia of a Box -->
-    <xacro:macro name="box_inertia" params="mass x y z">
-        <inertia ixx="${mass*(y*y+z*z)/12}" ixy = "0" ixz = "0"
-            iyy="${mass*(x*x+z*z)/12}" iyz = "0" izz="${mass*(x*x+y*y)/12}" />
-    </xacro:macro>
     <!-- Physical Properties -->
-    <!-- PCB density ~ FR4 density (kg/m^3) -->
+    <!-- PCB density ~= FR4 density (kg/m^3) -->
+    <!-- PCB thickness (m) -->
     <xacro:property name="pcb_density" value="1850" />
-    <!-- Torso mass (kg) and x,y dimensions (m) -->
-    <xacro:property name="torso_mass" value="0.01" />
+    <xacro:property name="pcb_thickness_z" value="0.0015" />
+    <!-- Torso x,y dimensions (m) and mass (kg) -->
     <xacro:property name="torso_x" value="0.14" />
     <xacro:property name="torso_y" value="0.04" />
-    <!-- Leg mass (kg) and x,y dimensions (m) -->
-    <xacro:property name="leg_link_mass" value="0.0008" />
+    <xacro:property name="torso_mass"
+        value="${pcb_density * torso_x * torso_y * pcb_thickness_z}" />
+    <!-- Leg x,y dimensions (m) -->
     <xacro:property name="leg_link_x" value="0.02" />
     <xacro:property name="leg_link_y" value="0.03" />
+    <xacro:property name="leg_link_mass"
+        value="${pcb_density * leg_link_x * leg_link_y * pcb_thickness_z}" />
     <!-- Joint limits (rad) -->
     <xacro:property name="joint_upper_limit" value="1.5708" />
@@ -29,12 +23,10 @@
     <xacro:property name="joint_effort_limit" value="0.01" />
     <xacro:property name="joint_velocity_limit" value="0.01" />
-    <!-- Joint damping (b = N*s/m) and spring constant (k = N/m) -->
+    <!-- Joint damping (N*m*s/rad) and friction (N*m) -->
     <xacro:property name="joint_damping" value="0.00003" />
     <xacro:property name="joint_friction" value="0.001" />
-    <!-- PCB thickness (m) -->
-    <xacro:property name="pcb_thickness_z" value="0.0005" />
-    <!-- Link Gazebo properties -->
-    <!-- Contact stiffness (kp) -->
-    <!-- Contact damping (kp) -->
+    <!-- Gazebo Properties -->
+    <!-- Link contact stiffness (kp) -->
+    <!-- Link contact damping (kp) -->
     <xacro:property name="link_kp" value="1000.0" />
     <xacro:property name="link_kd" value="1000.0" />
@@ -50,4 +42,10 @@
         <color rgba="0.98 0.41 0.055 1" />
     </material>
+    <!-- Equation Macros -->
+    <!-- Calculate Moment of Inertia of a Box -->
+    <xacro:macro name="box_inertia" params="mass x y z">
+        <inertia ixx="${mass*(y*y+z*z)/12}" ixy = "0" ixz = "0"
+            iyy="${mass*(x*x+z*z)/12}" iyz = "0" izz="${mass*(x*x+y*y)/12}" />
+    </xacro:macro>
     <!-- Base and Torso Definition -->
     <xacro:macro name="millihex_torso" params="color">

Commit message: verified torso_mass and leg_link_mass xacro property. verified moment of inertia macro equations.

File: robot/millihex_description.xacro (robot description, xacro)
@@ -7,15 +7,18 @@
     <!-- PCB thickness (m) -->
     <xacro:property name="pcb_density" value="1850" />
-    <xacro:property name="pcb_thickness_z" value="0.0015" />
-    <!-- Torso x,y dimensions (m) and mass (kg) -->
+    <xacro:property name="pcb_thickness_z" value="0.003" />
+    <!-- Torso Link x,y dimensions (m) and mass (kg) -->
     <xacro:property name="torso_x" value="0.14" />
     <xacro:property name="torso_y" value="0.04" />
     <xacro:property name="torso_mass"
         value="${pcb_density * torso_x * torso_y * pcb_thickness_z}" />
-    <!-- Leg x,y dimensions (m) -->
+    <!-- Leg Link x,y dimensions (m) and mass (kg) -->
     <xacro:property name="leg_link_x" value="0.02" />
     <xacro:property name="leg_link_y" value="0.03" />
     <xacro:property name="leg_link_mass"
         value="${pcb_density * leg_link_x * leg_link_y * pcb_thickness_z}" />
+    <!-- Massless Joint Link x,y dimensions (m) -->
+    <xacro:property name="joint_link_r" value="${pcb_thickness_z / 2}" />
+    <xacro:property name="joint_link_l" value="${leg_link_x}"
     <!-- Joint limits (rad) -->
     <xacro:property name="joint_upper_limit" value="1.5708" />

Commit message: created massless joint link.

File: robot/millihex_description.xacro (robot description, xacro)
@@ -20,5 +20,5 @@
     <!-- Massless Joint Link x,y dimensions (m) -->
     <xacro:property name="joint_link_r" value="${pcb_thickness_z / 2}" />
-    <xacro:property name="joint_link_l" value="${leg_link_x}"
+    <xacro:property name="joint_link_l" value="${leg_link_x}" />
     <!-- Joint limits (rad) -->
     <xacro:property name="joint_upper_limit" value="1.5708" />

Commit message: created fake joint link definition.

File: robot/millihex_description.xacro (robot description, xacro)
@@ -18,7 +18,7 @@
     <xacro:property name="leg_link_mass"
         value="${pcb_density * leg_link_x * leg_link_y * pcb_thickness_z}" />
-    <!-- Massless Joint Link x,y dimensions (m) -->
-    <xacro:property name="joint_link_r" value="${pcb_thickness_z / 2}" />
-    <xacro:property name="joint_link_l" value="${leg_link_x}"
+    <!-- Fake Joint Link r,l dimensions (m) -->
+    <xacro:property name="fake_joint_link_r" value="${pcb_thickness_z / 2}" />
+    <xacro:property name="fake_joint_link_l" value="${leg_link_x}" />
     <!-- Joint limits (rad) -->
     <xacro:property name="joint_upper_limit" value="1.5708" />
@@ -51,9 +51,9 @@
             iyy="${mass*(x*x+z*z)/12}" iyz = "0" izz="${mass*(x*x+y*y)/12}" />
     </xacro:macro>
-    <!-- Base and Torso Definition -->
+    <!-- Torso Definition -->
     <xacro:macro name="millihex_torso" params="color">
-        <!-- Dummy link to support KDL -->
+        <!-- Dummy Base Link to support KDL -->
         <link name="base_link" />
-        <!-- Torso geometry without legs -->
+        <!-- Torso Geometry -->
         <link name="torso">
             <inertial>
@@ -91,8 +91,37 @@
         </joint>
     </xacro:macro>
+    <!-- Fake Joint Link Definition -->
+    <xacro:macro name="millihex_fake_joint_link"
+        params="leg_number link_number x_length y_length color">
+        <!-- Fake Joint Link Geometry -->
+        <link name="leg${leg_number}_link${link_number}">
+            <collision>
+                <origin xyz="-${x_length / 2} -${y_length / 2} 0" rpy="0 0 0" />
+                <geometry>
+                    <cylinder radius="${fake_joint_link_r}"
+                        length="${fake_joint_link_l}" />
+                </geometry>
+            </collision>
+            <visual>
+                <origin xyz="-${x_length / 2} -${y_length / 2} 0" rpy="0 0 0" />
+                <geometry>
+                    <box size="${x_length} ${y_length} ${pcb_thickness_z}" />
+                </geometry>
+                <material name="${color}"/>
+            </visual>
+        </link>
+        <!-- Gazebo properties -->
+        <gazebo reference="leg${leg_number}_link${link_number}">
+            <kp>${link_kp}</kp>
+            <kd>${link_kd}</kd>
+            <mu1>${link_mu1}</mu1>
+            <mu2>${link_mu2}</mu2>
+            <material>Gazebo/${color}</material>
+        </gazebo>
+    </xacro:macro>
     <!-- Leg Link Definition -->
     <xacro:macro name="millihex_leg_link"
         params="leg_number link_number x_length y_length color">
-        <!-- Leg geometry -->
+        <!-- Leg Link Geometry -->
         <link name="leg${leg_number}_link${link_number}">
             <inertial>
