Commit message: outlining link definitions.

File: robot/millihex_description.xacro (robot description, xacro)
@@ -16,6 +16,6 @@
         value="${pcb_density * (thorax_x * thorax_y * pcb_thickness_z)}" />  <!-- (kg) -->
     <!-- Coxa Properties -->
-    <xacro:property name="coxa_x" value="0.14" />     <!-- x length (m) -->
-    <xacro:property name="coxa_y" value="0.04" />     <!-- y length (m) -->
+    <xacro:property name="coxa_x" value="0.01" />     <!-- x length (m) -->
+    <xacro:property name="coxa_y" value="0.01" />     <!-- y length (m) -->
     <xacro:property name="coxa_kp" value="1000.0" />  <!-- contact stiffness -->
     <xacro:property name="coxa_kd" value="1000.0" />  <!-- contact damping -->
@@ -25,6 +25,6 @@
         value="${pcb_density * (coxa_x * coxa_y * pcb_thickness_z)}" />  <!-- (kg) -->
     <!-- Femur (Leg Link 1) Properties -->
-    <xacro:property name="leg_link_1_x" value="0.02" />     <!-- x length (m) -->
-    <xacro:property name="leg_link_1_y" value="0.03" />     <!-- y length (m) -->
+    <xacro:property name="leg_link_1_x" value="0.01" />     <!-- x length (m) -->
+    <xacro:property name="leg_link_1_y" value="0.05" />     <!-- y length (m) -->
     <xacro:property name="leg_link_1_kp" value="1000.0" />  <!-- contact stiffness -->
     <xacro:property name="leg_link_1_kd" value="1000.0" />  <!-- contact damping -->
@@ -34,6 +34,6 @@
         value="${pcb_density * (leg_link_1_x * leg_link_2_y * pcb_thickness_z)}" />  <!-- (kg) -->
     <!-- Tibia (Leg Link 2) Properties -->
-    <xacro:property name="leg_link_2_x" value="0.02" />     <!-- x length (m) -->
-    <xacro:property name="leg_link_2_y" value="0.03" />     <!-- y length (m) -->
+    <xacro:property name="leg_link_2_x" value="0.05" />     <!-- x length (m) -->
+    <xacro:property name="leg_link_2_y" value="0.01" />     <!-- y length (m) -->
     <xacro:property name="leg_link_2_kp" value="1000.0" />  <!-- contact stiffness -->
     <xacro:property name="leg_link_2_kd" value="1000.0" />  <!-- contact damping -->
@@ -43,6 +43,6 @@
         value="${pcb_density * (leg_link_2_x * leg_link_2_y * pcb_thickness_z)}" />  <!-- (kg) -->
     <!-- Tarsus (Leg Link 3) Properties -->
-    <xacro:property name="leg_link_3_x" value="0.02" />     <!-- x length (m) -->
-    <xacro:property name="leg_link_3_y" value="0.03" />     <!-- y length (m) -->
+    <xacro:property name="leg_link_3_x" value="0.01" />     <!-- x length (m) -->
+    <xacro:property name="leg_link_3_y" value="0.05" />     <!-- y length (m) -->
     <xacro:property name="leg_link_3_kp" value="1000.0" />  <!-- contact stiffness -->
     <xacro:property name="leg_link_3_kd" value="1000.0" />  <!-- contact damping -->
@@ -52,6 +52,6 @@
         value="${pcb_density * (leg_link_3_x * leg_link_3_y * pcb_thickness_z)}" />  <!-- (kg) -->
     <!-- Joint Link Properties -->
-    <xacro:property name="joint_link_r" value="${pcb_thickness_z / 2}" />  <!-- radius (m) -->
-    <xacro:property name="joint_link_l" value="${leg_link_x}" />           <!-- length (m) -->
+    <xacro:property name="joint_link_r" value="0.0015" />  <!-- radius (m) -->
+    <xacro:property name="joint_link_l" value="0.01" />    <!-- length (m) -->
     <!-- Revolute Joint Properties -->
     <xacro:property name="joint_upper_limit" value="1.5708" />   <!-- (rad) -->
@@ -117,4 +117,70 @@
         </joint>
     </xacro:macro>
+    <!-- Coxa Definition -->
+    <xacro:macro name="millihex_coxa" params="leg_number color">
+        <!-- Coxa Geometry -->
+        <link name="leg${leg_number}_coxa">
+            <inertial>
+                <origin xyz="0 0 ${pcb_thickness_z / 2}" rpy="0 0 0" />
+                <mass value="${coxa_mass}" />
+                <xacro:box_inertia mass="${coxa_mass}" x="${coxa_x}"
+                    y="${coxa_y}" z="${pcb_thickness_z}" />
+            </inertial>
+            <collision>
+                <origin xyz="0 0 0" rpy="0 0 0" />
+                <geometry>
+                    <box size="${coxa_x} ${coxa_y} ${pcb_thickness_z}" />
+                </geometry>
+            </collision>
+            <visual>
+                <origin xyz="0 0 0" rpy="0 0 0" />
+                <geometry>
+                    <box size="${coxa_x} ${coxa_y} ${pcb_thickness_z}" />
+                </geometry>
+                <material name="${color}"/>
+            </visual>
+        </link>
+        <!-- Gazebo properties -->
+        <gazebo reference="leg${leg_number}_coxa">
+            <kp>${coxa_kp}</kp>
+            <kd>${coxa_kd}</kd>
+            <mu1>${coxa_mu1}</mu1>
+            <mu2>${coxa_mu2}</mu2>
+            <material>Gazebo/${color}</material>
+        </gazebo>
+    </xacro:macro>
+    <!-- Femur (Leg Link 1) Definition -->
+    <xacro:macro name="millihex_leg_link_1" params="leg_number color">
+        <!-- Femur (Leg Link 1) Geometry -->
+        <link name="leg${leg_number}_link1">
+            <inertial>
+                <origin xyz="0 0 ${pcb_thickness_z / 2}" rpy="0 0 0" />
+                <mass value="${leg_link_1_mass}" />
+                <xacro:box_inertia mass="${leg_link_1_mass}" x="${leg_link_1_x}"
+                    y="${leg_link_1_y}" z="${pcb_thickness_z}" />
+            </inertial>
+            <collision>
+                <origin xyz="0 0 0" rpy="0 0 0" />
+                <geometry>
+                    <box size="${leg_link_1_x} ${leg_link_1_y} ${pcb_thickness_z}" />
+                </geometry>
+            </collision>
+            <visual>
+                <origin xyz="0 0 0" rpy="0 0 0" />
+                <geometry>
+                    <box size="${leg_link_1_x} ${leg_link_1_y} ${pcb_thickness_z}" />
+                </geometry>
+                <material name="${color}"/>
+            </visual>
+        </link>
+        <!-- Gazebo properties -->
+        <gazebo reference="leg${leg_number}_link1">
+            <kp>${leg_link_1_kp}</kp>
+            <kd>${leg_link_1_kd}</kd>
+            <mu1>${leg_link_1_mu1}</mu1>
+            <mu2>${leg_link_1_mu2}</mu2>
+            <material>Gazebo/${color}</material>
+        </gazebo>
+    </xacro:macro>
     <!-- Joint Link Definition -->
     <xacro:macro name="millihex_joint_link" params="leg_number link_number color">
@@ -122,14 +188,13 @@
         <link name="leg${leg_number}_joint_link${link_number}">
             <collision>
-                <origin xyz="-${x_length / 2} -${y_length / 2} 0" rpy="0 0 0" />
-                <geometry>
-                    <cylinder radius="${fake_joint_link_r}"
-                        length="${fake_joint_link_l}" />
-                </geometry>
-            </collision>
-            <visual>
-                <origin xyz="-${x_length / 2} -${y_length / 2} 0" rpy="0 0 0" />
-                <geometry>
-                    <box size="${x_length} ${y_length} ${pcb_thickness_z}" />
+                <origin xyz="0 0 0" rpy="0 0 0" />
+                <geometry>
+                    <cylinder radius="${joint_link_r}" length="${joint_link_l}" />
+                </geometry>
+            </collision>
+            <visual>
+                <origin xyz="0 0 0" rpy="0 0 0" />
+                <geometry>
+                    <cylinder radius="${joint_link_r}" length="${joint_link_l}" />
                 </geometry>
                 <material name="${color}"/>
@@ -137,43 +202,5 @@
         </link>
         <!-- Gazebo properties -->
-        <gazebo reference="leg${leg_number}_link${link_number}">
-            <kp>${link_kp}</kp>
-            <kd>${link_kd}</kd>
-            <mu1>${link_mu1}</mu1>
-            <mu2>${link_mu2}</mu2>
-            <material>Gazebo/${color}</material>
-        </gazebo>
-    </xacro:macro>
-    <!-- Leg Link Definition -->
-    <xacro:macro name="millihex_leg_link"
-        params="leg_number link_number x_length y_length color">
-        <!-- Leg Link Geometry -->
-        <link name="leg${leg_number}_link${link_number}">
-            <inertial>
-                <origin xyz="0 0 ${pcb_thickness_z / 2}" rpy="0 0 0" />
-                <mass value="${leg_link_mass}" />
-                <xacro:box_inertia mass="${leg_link_mass}" x="${x_length}"
-                    y="${y_length}" z="${pcb_thickness_z}" />
-            </inertial>
-            <collision>
-                <origin xyz="-${x_length / 2} -${y_length / 2} 0" rpy="0 0 0" />
-                <geometry>
-                    <box size="${x_length} ${y_length} ${pcb_thickness_z}" />
-                </geometry>
-            </collision>
-            <visual>
-                <origin xyz="-${x_length / 2} -${y_length / 2} 0" rpy="0 0 0" />
-                <geometry>
-                    <box size="${x_length} ${y_length} ${pcb_thickness_z}" />
-                </geometry>
-                <material name="${color}"/>
-            </visual>
-        </link>
-        <!-- Gazebo properties -->
-        <gazebo reference="leg${leg_number}_link${link_number}">
-            <kp>${link_kp}</kp>
-            <kd>${link_kd}</kd>
-            <mu1>${link_mu1}</mu1>
-            <mu2>${link_mu2}</mu2>
+        <gazebo reference="leg${leg_number}_joint_link${link_number}">
             <material>Gazebo/${color}</material>
         </gazebo>
@@ -219,6 +246,6 @@
     <!-- Assemble Body -->
     <xacro:macro name="millihex_body" params="">
-        <!-- Call Torso xacro -->
-        <xacro:millihex_torso color="Orange" />
+        <!-- Call Thorax xacro -->
+        <xacro:millihex_thorax color="Orange" />
         <!-- Leg 1-->
         <xacro:millihex_leg leg_number="1" />

Commit message: torso, coxa, and link1 spawn ok in gazebo. errors with joint position controllers.

File: robot/millihex_description.xacro (robot description, xacro)
@@ -3,4 +3,12 @@
 <!-- rosrun xacro xacro millihex_description.xacro > millihex_description.urdf -->
 <robot name="millihex" xmlns:xacro="http://www.ros.org/wiki/xacro">
+    <!-- Gazebo Control Library -->
+    <xacro:macro name="millihex_control" params="namespace">
+        <gazebo>
+            <plugin name="gazebo_ros_control" filename="libgazebo_ros_control.so">
+                <robotNamespace>/${namespace}</robotNamespace>
+            </plugin>
+        </gazebo>
+    </xacro:macro>
     <!-- PCB Properties -->
     <xacro:property name="pcb_density" value="1850" />       <!-- FR4 density (kg/m^3) -->
@@ -51,4 +59,11 @@
     <xacro:property name="leg_link_3_mass"
         value="${pcb_density * (leg_link_3_x * leg_link_3_y * pcb_thickness_z)}" />  <!-- (kg) -->
+    <!-- Thorax Leg Joint Attachment Positions -->
+    <xacro:property name="leg_spacing" value="${(2 * coxa_x) + leg_link_2_x}" />
+    <xacro:property name="frontal_leg_x" value="${(thorax_x / 2) - (coxa_x / 2)}" />
+    <xacro:property name="medial_leg_x" value="${frontal_leg_x - leg_spacing}" />
+    <xacro:property name="hind_leg_x" value="${medial_leg_x - leg_spacing}" />
+    <xacro:property name="right_side_y" value="${thorax_y / 2}" />
+    <xacro:property name="left_side_y" value="${-(thorax_y / 2)}" />
     <!-- Joint Link Properties -->
     <xacro:property name="joint_link_r" value="0.0015" />  <!-- radius (m) -->
@@ -71,5 +86,4 @@
         <color rgba="0.98 0.41 0.055 1.0" />
     </material>
-    <!-- Equation Macros -->
     <!-- Calculate Moment of Inertia of a Box -->
     <xacro:macro name="box_inertia" params="mass x y z">
@@ -206,5 +220,5 @@
         </gazebo>
     </xacro:macro>
-    <!-- Leg Joint Transmission -->
+    <!-- Joint Transmission -->
     <xacro:macro name="leg_transmission" params="leg_number joint_number">
         <transmission name="leg${leg_number}_joint${joint_number}_tran">
@@ -225,14 +239,12 @@
     <!-- Assemble Leg -->
     <xacro:macro name="millihex_leg" params="leg_number">
-        <!-- Link 0 (shoulder link), horizontally oriented -->
-        <xacro:millihex_leg_link leg_number="${leg_number}" link_number="0"
-            x_length="${leg_link_x}" y_length="${leg_link_y}" color="Black" />
-        <!-- Link 1, vertically oriented -->
-        <xacro:millihex_leg_link leg_number="${leg_number}" link_number="1"
-            x_length="${leg_link_y}" y_length="${leg_link_x}" color="Orange" />
+        <!-- Coxa -->
+        <xacro:millihex_coxa leg_number="${leg_number}" color="Black" />
+        <!-- Coxa to Femur Joint Link (Joint Link 1) -->
+        <xacro:millihex_joint_link leg_number="${leg_number}" link_number="1" color="Cyan" />
+        <!-- leg#_joint1 -->
         <joint name="leg${leg_number}_joint1" type="revolute">
-            <parent link="leg${leg_number}_link0" />
-            <child link="leg${leg_number}_link1" />
-            <origin xyz="0 -${leg_link_y} 0" rpy="0 0 0" />
+            <parent link="leg${leg_number}_coxa" />
+            <child link="leg${leg_number}_joint_link1" />
             <dynamics damping="${joint_damping}" friction="${joint_friction}" />
             <limit lower="${joint_lower_limit}"
@@ -243,27 +255,26 @@
         </joint>
         <xacro:leg_transmission leg_number="${leg_number}" joint_number="1" />
+        <!-- Femur (Leg Link 1) -->
+        <xacro:millihex_leg_link_1 leg_number="${leg_number}" color="Orange" />
+        <!-- leg#_fixed_joint1 -->
+        <joint name="leg${leg_number}_fixed_joint1" type="fixed">
+            <parent link="leg${leg_number}_joint_link1" />
+            <child link="leg${leg_number}_link1" />
+            <origin xyz="0 0 0" rpy="0 0 0" />
+        </joint>
     </xacro:macro>
     <!-- Assemble Body -->
     <xacro:macro name="millihex_body" params="">
-        <!-- Call Thorax xacro -->
+        <!-- Thorax -->
         <xacro:millihex_thorax color="Orange" />
-        <!-- Leg 1-->
+        <!-- Leg 1 -->
         <xacro:millihex_leg leg_number="1" />
-        <!-- Leg 1, Joint 0 (fixed, shoulder joint)-->
-        <joint name="leg1_joint0" type="fixed">
-            <parent link="torso" />
-            <child link="leg1_link0" />
-            <origin xyz="${torso_x / 2} -${torso_y / 2} 0" rpy="0 0 0" />
-        </joint>
-    </xacro:macro>
-    <!-- Add Gazebo Control Library -->
-    <xacro:macro name="millihex_control" params="namespace">
-        <gazebo>
-            <plugin name="gazebo_ros_control" filename="libgazebo_ros_control.so">
-                <robotNamespace>/${namespace}</robotNamespace>
-            </plugin>
-        </gazebo>
-    </xacro:macro>
-    <!-- Build Robot and Gazebo Control Library -->
+        <joint name="leg1_coxa_joint" type="fixed">
+            <parent link="thorax" />
+            <child link="leg1_coxa" />
+            <origin xyz="${frontal_leg_x} ${right_side_y} 0" rpy="0 0 0" />
+        </joint>
+    </xacro:macro>
+    <!-- Assemble Robot -->
     <xacro:millihex_body />
     <xacro:millihex_control namespace="millihex" />

Commit message: constructed femur link for leg 1.

File: robot/millihex_description.xacro (robot description, xacro)
@@ -64,6 +64,6 @@
     <xacro:property name="medial_leg_x" value="${frontal_leg_x - leg_spacing}" />
     <xacro:property name="hind_leg_x" value="${medial_leg_x - leg_spacing}" />
-    <xacro:property name="right_side_y" value="${thorax_y / 2}" />
-    <xacro:property name="left_side_y" value="${-(thorax_y / 2)}" />
+    <xacro:property name="right_side_y" value="${(thorax_y / 2) + (coxa_y / 2)}" />
+    <xacro:property name="left_side_y" value="${-((thorax_y / 2) + (coxa_y / 2))}" />
     <!-- Joint Link Properties -->
     <xacro:property name="joint_link_r" value="0.0015" />  <!-- radius (m) -->
@@ -77,7 +77,4 @@
     <xacro:property name="joint_friction" value="0.0" />         <!-- friction (N*m) -->
     <!-- Color Definitions -->
-    <material name="Cyan">
-        <color rgba="0.0 1.0 1.0 1.0" />
-    </material>
     <material name="Black">
         <color rgba="0.0 0.0 0.0 1.0" />
@@ -85,4 +82,7 @@
     <material name="Orange">
         <color rgba="0.98 0.41 0.055 1.0" />
+    </material>
+    <material name="White">
+        <color rgba="0.0 0.0 0.0 0.0" />
     </material>
     <!-- Calculate Moment of Inertia of a Box -->
@@ -198,5 +198,6 @@
     </xacro:macro>
     <!-- Joint Link Definition -->
-    <xacro:macro name="millihex_joint_link" params="leg_number link_number color">
+    <xacro:macro name="millihex_joint_link"
+        params="leg_number link_number yaw color">
         <!-- Joint Link Geometry -->
         <link name="leg${leg_number}_joint_link${link_number}">
@@ -208,5 +209,5 @@
             </collision>
             <visual>
-                <origin xyz="0 0 0" rpy="0 0 0" />
+                <origin xyz="0 0 0" rpy="0 ${pi / 2} ${yaw}" />
                 <geometry>
                     <cylinder radius="${joint_link_r}" length="${joint_link_l}" />
@@ -242,9 +243,11 @@
         <xacro:millihex_coxa leg_number="${leg_number}" color="Black" />
         <!-- Coxa to Femur Joint Link (Joint Link 1) -->
-        <xacro:millihex_joint_link leg_number="${leg_number}" link_number="1" color="Cyan" />
+        <xacro:millihex_joint_link leg_number="${leg_number}" link_number="1"
+            yaw="0.0" color="White" />
         <!-- leg#_joint1 -->
         <joint name="leg${leg_number}_joint1" type="revolute">
             <parent link="leg${leg_number}_coxa" />
             <child link="leg${leg_number}_joint_link1" />
+            <origin xyz="0 ${(coxa_y / 2) + (joint_link_r)} 0" rpy="0 0 0" />
             <dynamics damping="${joint_damping}" friction="${joint_friction}" />
             <limit lower="${joint_lower_limit}"
@@ -261,5 +264,5 @@
             <parent link="leg${leg_number}_joint_link1" />
             <child link="leg${leg_number}_link1" />
-            <origin xyz="0 0 0" rpy="0 0 0" />
+            <origin xyz="0 ${(leg_link_1_y / 2) + (joint_link_r)} 0" rpy="0 0 0" />
         </joint>
     </xacro:macro>
