Commit message: added all legs with new dimensions and joint links.

File: robot/millihex_description.xacro (robot description, xacro)
@@ -15,6 +15,6 @@
     <xacro:property name="pcb_thickness_z" value="0.003" />  <!-- PCB thickness (m) -->
     <!-- Thorax Properties -->
-    <xacro:property name="thorax_x" value="0.20" />     <!-- x length (m) -->
-    <xacro:property name="thorax_y" value="0.03" />     <!-- y length (m) -->
+    <xacro:property name="thorax_x" value="0.25" />     <!-- x length (m) -->
+    <xacro:property name="thorax_y" value="0.02" />     <!-- y length (m) -->
     <xacro:property name="thorax_kp" value="1000.0" />  <!-- contact stiffness -->
     <xacro:property name="thorax_kd" value="1000.0" />  <!-- contact damping -->
@@ -70,10 +70,10 @@
     <xacro:property name="joint_link_l" value="0.01" />    <!-- length (m) -->
     <!-- Revolute Joint Properties -->
-    <xacro:property name="joint_upper_limit" value="1.5708" />   <!-- (rad) -->
-    <xacro:property name="joint_lower_limit" value="-1.5708" />  <!-- (rad) -->
-    <xacro:property name="joint_effort_limit" value="0.1" />     <!-- (rad/s) -->
-    <xacro:property name="joint_velocity_limit" value="0.1" />   <!-- (rad/s) -->
-    <xacro:property name="joint_damping" value="0.0" />          <!-- damping (N*m*s/rad)-->
-    <xacro:property name="joint_friction" value="0.0" />         <!-- friction (N*m) -->
+    <xacro:property name="joint_upper_limit" value="${pi / 2}" />   <!-- (rad) -->
+    <xacro:property name="joint_lower_limit" value="${-pi / 2}" />  <!-- (rad) -->
+    <xacro:property name="joint_effort_limit" value="0.1" />        <!-- (rad/s) -->
+    <xacro:property name="joint_velocity_limit" value="0.1" />      <!-- (rad/s) -->
+    <xacro:property name="joint_damping" value="0.0" />   <!-- damping (N*m*s/rad)-->
+    <xacro:property name="joint_friction" value="0.0" />  <!-- friction (N*m) -->
     <!-- Color Definitions -->
     <material name="Black">
@@ -194,4 +194,70 @@
             <mu1>${leg_link_1_mu1}</mu1>
             <mu2>${leg_link_1_mu2}</mu2>
+            <material>Gazebo/${color}</material>
+        </gazebo>
+    </xacro:macro>
+    <!-- Tibia (Leg Link 2) Definition -->
+    <xacro:macro name="millihex_leg_link_2" params="leg_number color">
+        <!-- Tibia (Leg Link 2) Geometry -->
+        <link name="leg${leg_number}_link2">
+            <inertial>
+                <origin xyz="0 0 ${pcb_thickness_z / 2}" rpy="0 0 0" />
+                <mass value="${leg_link_2_mass}" />
+                <xacro:box_inertia mass="${leg_link_2_mass}" x="${leg_link_2_x}"
+                    y="${leg_link_2_y}" z="${pcb_thickness_z}" />
+            </inertial>
+            <collision>
+                <origin xyz="0 0 0" rpy="0 0 0" />
+                <geometry>
+                    <box size="${leg_link_2_x} ${leg_link_2_y} ${pcb_thickness_z}" />
+                </geometry>
+            </collision>
+            <visual>
+                <origin xyz="0 0 0" rpy="0 0 0" />
+                <geometry>
+                    <box size="${leg_link_2_x} ${leg_link_2_y} ${pcb_thickness_z}" />
+                </geometry>
+                <material name="${color}"/>
+            </visual>
+        </link>
+        <!-- Gazebo properties -->
+        <gazebo reference="leg${leg_number}_link2">
+            <kp>${leg_link_2_kp}</kp>
+            <kd>${leg_link_2_kd}</kd>
+            <mu1>${leg_link_2_mu1}</mu1>
+            <mu2>${leg_link_2_mu2}</mu2>
+            <material>Gazebo/${color}</material>
+        </gazebo>
+    </xacro:macro>
+    <!-- Tarsus (Leg Link 3) Definition -->
+    <xacro:macro name="millihex_leg_link_3" params="leg_number color">
+        <!-- Tarsus (Leg Link 3) Geometry -->
+        <link name="leg${leg_number}_link3">
+            <inertial>
+                <origin xyz="0 0 ${pcb_thickness_z / 2}" rpy="0 0 0" />
+                <mass value="${leg_link_3_mass}" />
+                <xacro:box_inertia mass="${leg_link_3_mass}" x="${leg_link_3_x}"
+                    y="${leg_link_3_y}" z="${pcb_thickness_z}" />
+            </inertial>
+            <collision>
+                <origin xyz="0 0 0" rpy="0 0 0" />
+                <geometry>
+                    <box size="${leg_link_3_x} ${leg_link_3_y} ${pcb_thickness_z}" />
+                </geometry>
+            </collision>
+            <visual>
+                <origin xyz="0 0 0" rpy="0 0 0" />
+                <geometry>
+                    <box size="${leg_link_3_x} ${leg_link_3_y} ${pcb_thickness_z}" />
+                </geometry>
+                <material name="${color}"/>
+            </visual>
+        </link>
+        <!-- Gazebo properties -->
+        <gazebo reference="leg${leg_number}_link3">
+            <kp>${leg_link_3_kp}</kp>
+            <kd>${leg_link_3_kd}</kd>
+            <mu1>${leg_link_3_mu1}</mu1>
+            <mu2>${leg_link_3_mu2}</mu2>
             <material>Gazebo/${color}</material>
         </gazebo>
@@ -266,4 +332,53 @@
             <origin xyz="0 ${(leg_link_1_y / 2) + (joint_link_r)} 0" rpy="0 0 0" />
         </joint>
+        <!-- Femur to Tibia Joint Link (Joint Link 2) -->
+        <xacro:millihex_joint_link leg_number="${leg_number}" link_number="2"
+            yaw="${pi / 2}" color="White" />
+        <!-- leg#_joint2 -->
+        <joint name="leg${leg_number}_joint2" type="revolute">
+            <parent link="leg${leg_number}_link1" />
+            <child link="leg${leg_number}_joint_link2" />
+            <origin xyz="${-((leg_link_1_x / 2) + (joint_link_r))}
+                ${(leg_link_1_y / 2) - (joint_link_l / 2)} 0" rpy="0 0 0" />
+            <dynamics damping="${joint_damping}" friction="${joint_friction}" />
+            <limit lower="${joint_lower_limit}"
+                   upper="${joint_upper_limit}"
+                   effort="${joint_effort_limit}"
+                   velocity="${joint_velocity_limit}" />
+            <axis xyz="0 1 0" />
+        </joint>
+        <xacro:leg_transmission leg_number="${leg_number}" joint_number="2" />
+        <!-- Tibia (Leg Link 2) -->
+        <xacro:millihex_leg_link_2 leg_number="${leg_number}" color="Black" />
+        <!-- leg#_fixed_joint2 -->
+        <joint name="leg${leg_number}_fixed_joint2" type="fixed">
+            <parent link="leg${leg_number}_joint_link2" />
+            <child link="leg${leg_number}_link2" />
+            <origin xyz="${-((leg_link_2_x / 2) + (joint_link_r))} 0 0" rpy="0 0 0" />
+        </joint>
+        <!-- Tibia to Tarsus Joint Link (Joint Link 3) -->
+        <xacro:millihex_joint_link leg_number="${leg_number}" link_number="3"
+            yaw="0.0" color="White" />
+        <!-- leg#_joint3 -->
+        <joint name="leg${leg_number}_joint3" type="revolute">
+            <parent link="leg${leg_number}_link2" />
+            <child link="leg${leg_number}_joint_link3" />
+            <origin xyz="${-(leg_link_2_x / 2) + (joint_link_l / 2)} ${(leg_link_2_y / 2) + (joint_link_r)} 0" rpy="0 0 0" />
+            <dynamics damping="${joint_damping}" friction="${joint_friction}" />
+            <limit lower="${joint_lower_limit}"
+                   upper="${joint_upper_limit}"
+                   effort="${joint_effort_limit}"
+                   velocity="${joint_velocity_limit}" />
+            <axis xyz="1 0 0" />
+        </joint>
+        <xacro:leg_transmission leg_number="${leg_number}" joint_number="3" />
+        <!-- Tarsus (Leg Link 3) -->
+        <xacro:millihex_leg_link_3 leg_number="${leg_number}" color="Orange" />
+        <!-- leg#_fixed_joint3 -->
+        <joint name="leg${leg_number}_fixed_joint3" type="fixed">
+            <parent link="leg${leg_number}_joint_link3" />
+            <child link="leg${leg_number}_link3" />
+            <origin xyz="0 ${(leg_link_3_y / 2) + (joint_link_r)} 0" rpy="0 0 0" />
+        </joint>
     </xacro:macro>
     <!-- Assemble Body -->
@@ -278,4 +393,39 @@
             <origin xyz="${frontal_leg_x} ${right_side_y} 0" rpy="0 0 0" />
         </joint>
+        <!-- Leg 2 -->
+        <xacro:millihex_leg leg_number="2" />
+        <joint name="leg2_coxa_joint" type="fixed">
+            <parent link="thorax" />
+            <child link="leg2_coxa" />
+            <origin xyz="${medial_leg_x} ${right_side_y} 0" rpy="0 0 0" />
+        </joint>
+        <!-- Leg 3 -->
+        <xacro:millihex_leg leg_number="3" />
+        <joint name="leg3_coxa_joint" type="fixed">
+            <parent link="thorax" />
+            <child link="leg3_coxa" />
+            <origin xyz="${hind_leg_x} ${right_side_y} 0" rpy="0 0 0" />
+        </joint>
+        <!-- Leg 4 -->
+        <xacro:millihex_leg leg_number="4" />
+        <joint name="leg4_coxa_joint" type="fixed">
+            <parent link="thorax" />
+            <child link="leg4_coxa" />
+            <origin xyz="${frontal_leg_x} ${left_side_y} 0" rpy="${pi} 0 0" />
+        </joint>
+        <!-- Leg 5 -->
+        <xacro:millihex_leg leg_number="5" />
+        <joint name="leg5_coxa_joint" type="fixed">
+            <parent link="thorax" />
+            <child link="leg5_coxa" />
+            <origin xyz="${medial_leg_x} ${left_side_y} 0" rpy="${pi} 0 0" />
+        </joint>
+        <!-- Leg 6 -->
+        <xacro:millihex_leg leg_number="6" />
+        <joint name="leg6_coxa_joint" type="fixed">
+            <parent link="thorax" />
+            <child link="leg6_coxa" />
+            <origin xyz="${hind_leg_x} ${left_side_y} 0" rpy="${pi} 0 0" />
+        </joint>
     </xacro:macro>
     <!-- Assemble Robot -->

Commit message: inverted joint axis direction.

File: robot/millihex_description.xacro (robot description, xacro)
@@ -321,5 +321,5 @@
                    effort="${joint_effort_limit}"
                    velocity="${joint_velocity_limit}" />
-            <axis xyz="1 0 0" />
+            <axis xyz="-1 0 0" />
         </joint>
         <xacro:leg_transmission leg_number="${leg_number}" joint_number="1" />
@@ -346,5 +346,5 @@
                    effort="${joint_effort_limit}"
                    velocity="${joint_velocity_limit}" />
-            <axis xyz="0 1 0" />
+            <axis xyz="0 -1 0" />
         </joint>
         <xacro:leg_transmission leg_number="${leg_number}" joint_number="2" />
@@ -364,5 +364,6 @@
             <parent link="leg${leg_number}_link2" />
             <child link="leg${leg_number}_joint_link3" />
-            <origin xyz="${-(leg_link_2_x / 2) + (joint_link_l / 2)} ${(leg_link_2_y / 2) + (joint_link_r)} 0" rpy="0 0 0" />
+            <origin xyz="${-(leg_link_2_x / 2) + (joint_link_l / 2)}
+                ${(leg_link_2_y / 2) + (joint_link_r)} 0" rpy="0 0 0" />
             <dynamics damping="${joint_damping}" friction="${joint_friction}" />
             <limit lower="${joint_lower_limit}"
@@ -370,5 +371,5 @@
                    effort="${joint_effort_limit}"
                    velocity="${joint_velocity_limit}" />
-            <axis xyz="1 0 0" />
+            <axis xyz="-1 0 0" />
         </joint>
         <xacro:leg_transmission leg_number="${leg_number}" joint_number="3" />

Commit message: simplified xacro by getting rid of extra link properties to make debugging easier. added joint link inertias which were previously nonexistent. testing different pid properties in millihex_control. created millihex_control_autogen file to make changing pid values for all joints faster.

File: robot/millihex_description.xacro (robot description, xacro)
@@ -17,8 +17,4 @@
     <xacro:property name="thorax_x" value="0.25" />     <!-- x length (m) -->
     <xacro:property name="thorax_y" value="0.02" />     <!-- y length (m) -->
-    <xacro:property name="thorax_kp" value="1000.0" />  <!-- contact stiffness -->
-    <xacro:property name="thorax_kd" value="1000.0" />  <!-- contact damping -->
-    <xacro:property name="thorax_mu1" value="10.0" />   <!-- friction coef 1 -->
-    <xacro:property name="thorax_mu2" value="10.0" />   <!-- friction coef 2 -->
     <xacro:property name="thorax_mass"
         value="${pcb_density * (thorax_x * thorax_y * pcb_thickness_z)}" />  <!-- (kg) -->
@@ -26,8 +22,4 @@
     <xacro:property name="coxa_x" value="0.01" />     <!-- x length (m) -->
     <xacro:property name="coxa_y" value="0.01" />     <!-- y length (m) -->
-    <xacro:property name="coxa_kp" value="1000.0" />  <!-- contact stiffness -->
-    <xacro:property name="coxa_kd" value="1000.0" />  <!-- contact damping -->
-    <xacro:property name="coxa_mu1" value="10.0" />   <!-- friction coef 1 -->
-    <xacro:property name="coxa_mu2" value="10.0" />   <!-- friction coef 2 -->
     <xacro:property name="coxa_mass"
         value="${pcb_density * (coxa_x * coxa_y * pcb_thickness_z)}" />  <!-- (kg) -->
@@ -35,8 +27,4 @@
     <xacro:property name="leg_link_1_x" value="0.01" />     <!-- x length (m) -->
     <xacro:property name="leg_link_1_y" value="0.05" />     <!-- y length (m) -->
-    <xacro:property name="leg_link_1_kp" value="1000.0" />  <!-- contact stiffness -->
-    <xacro:property name="leg_link_1_kd" value="1000.0" />  <!-- contact damping -->
-    <xacro:property name="leg_link_1_mu1" value="10.0" />   <!-- friction coef 1 -->
-    <xacro:property name="leg_link_1_mu2" value="10.0" />   <!-- friction coef 2 -->
     <xacro:property name="leg_link_1_mass"
         value="${pcb_density * (leg_link_1_x * leg_link_2_y * pcb_thickness_z)}" />  <!-- (kg) -->
@@ -44,8 +32,4 @@
     <xacro:property name="leg_link_2_x" value="0.05" />     <!-- x length (m) -->
     <xacro:property name="leg_link_2_y" value="0.01" />     <!-- y length (m) -->
-    <xacro:property name="leg_link_2_kp" value="1000.0" />  <!-- contact stiffness -->
-    <xacro:property name="leg_link_2_kd" value="1000.0" />  <!-- contact damping -->
-    <xacro:property name="leg_link_2_mu1" value="10.0" />   <!-- friction coef 1 -->
-    <xacro:property name="leg_link_2_mu2" value="10.0" />   <!-- friction coef 2 -->
     <xacro:property name="leg_link_2_mass"
         value="${pcb_density * (leg_link_2_x * leg_link_2_y * pcb_thickness_z)}" />  <!-- (kg) -->
@@ -53,10 +37,16 @@
     <xacro:property name="leg_link_3_x" value="0.01" />     <!-- x length (m) -->
     <xacro:property name="leg_link_3_y" value="0.05" />     <!-- y length (m) -->
-    <xacro:property name="leg_link_3_kp" value="1000.0" />  <!-- contact stiffness -->
-    <xacro:property name="leg_link_3_kd" value="1000.0" />  <!-- contact damping -->
-    <xacro:property name="leg_link_3_mu1" value="10.0" />   <!-- friction coef 1 -->
-    <xacro:property name="leg_link_3_mu2" value="10.0" />   <!-- friction coef 2 -->
     <xacro:property name="leg_link_3_mass"
         value="${pcb_density * (leg_link_3_x * leg_link_3_y * pcb_thickness_z)}" />  <!-- (kg) -->
+    <!-- Joint Link Properties -->
+    <xacro:property name="joint_link_r" value="0.0015" />  <!-- radius (m) -->
+    <xacro:property name="joint_link_l" value="0.01" />    <!-- length (m) -->
+    <xacro:property name="joint_link_mass"
+        value="${pcb_density * (pi * (joint_link_r * joint_link_r) * joint_link_l)}" />  <!-- (kg) -->
+    <!-- Revolute Joint Properties -->
+    <xacro:property name="joint_upper_limit" value="${pi / 2}" />   <!-- (rad) -->
+    <xacro:property name="joint_lower_limit" value="${-pi / 2}" />  <!-- (rad) -->
+    <xacro:property name="joint_effort_limit" value="0.1" />        <!-- (N*m) -->
+    <xacro:property name="joint_velocity_limit" value="${pi / 4}" />      <!-- (rad/s) -->
     <!-- Thorax Leg Joint Attachment Positions -->
     <xacro:property name="leg_spacing" value="${(2 * coxa_x) + leg_link_2_x}" />
@@ -66,14 +56,4 @@
     <xacro:property name="right_side_y" value="${(thorax_y / 2) + (coxa_y / 2)}" />
     <xacro:property name="left_side_y" value="${-((thorax_y / 2) + (coxa_y / 2))}" />
-    <!-- Joint Link Properties -->
-    <xacro:property name="joint_link_r" value="0.0015" />  <!-- radius (m) -->
-    <xacro:property name="joint_link_l" value="0.01" />    <!-- length (m) -->
-    <!-- Revolute Joint Properties -->
-    <xacro:property name="joint_upper_limit" value="${pi / 2}" />   <!-- (rad) -->
-    <xacro:property name="joint_lower_limit" value="${-pi / 2}" />  <!-- (rad) -->
-    <xacro:property name="joint_effort_limit" value="0.1" />        <!-- (rad/s) -->
-    <xacro:property name="joint_velocity_limit" value="0.1" />      <!-- (rad/s) -->
-    <xacro:property name="joint_damping" value="0.0" />   <!-- damping (N*m*s/rad)-->
-    <xacro:property name="joint_friction" value="0.0" />  <!-- friction (N*m) -->
     <!-- Color Definitions -->
     <material name="Black">
@@ -88,6 +68,13 @@
     <!-- Calculate Moment of Inertia of a Box -->
     <xacro:macro name="box_inertia" params="mass x y z">
-        <inertia ixx="${mass*(y*y+z*z)/12}" ixy = "0" ixz = "0"
-            iyy="${mass*(x*x+z*z)/12}" iyz = "0" izz="${mass*(x*x+y*y)/12}" />
+        <inertia ixx="${(1 / 12) * mass * ((y * y) + (z * z))}" ixy = "0" ixz = "0"
+                 iyy="${(1 / 12) * mass * ((x * x) + (z * z))}" iyz = "0"
+                 izz="${(1 / 12) * mass * ((x * x) + (y * y))}" />
+    </xacro:macro>
+    <!-- Calculate Moment of Inertia of a Cylinder -->
+    <xacro:macro name="cylinder_inerta" params="mass r l">
+        <inertia ixx="${(1 / 12) * mass * (l * l)}" ixy = "0" ixz = "0"
+                 iyy="${(1 / 12) * mass * (l * l)}" iyz = "0"
+                 izz="${(1 / 2) * mass * (r * r)}" />
     </xacro:macro>
     <!-- Thorax Definition -->
@@ -98,5 +85,5 @@
         <link name="thorax">
             <inertial>
-                <origin xyz="0 0 ${pcb_thickness_z / 2}" rpy="0 0 0" />
+                <origin xyz="0 0 0" rpy="0 0 0" />
                 <mass value="${thorax_mass}" />
                 <xacro:box_inertia mass="${thorax_mass}" x="${thorax_x}"
@@ -119,8 +106,4 @@
         <!-- Gazebo properties -->
         <gazebo reference="thorax">
-            <kp>${thorax_kp}</kp>
-            <kd>${thorax_kd}</kd>
-            <mu1>${thorax_mu1}</mu1>
-            <mu2>${thorax_mu2}</mu2>
             <material>Gazebo/${color}</material>
         </gazebo>
@@ -136,5 +119,5 @@
         <link name="leg${leg_number}_coxa">
             <inertial>
-                <origin xyz="0 0 ${pcb_thickness_z / 2}" rpy="0 0 0" />
+                <origin xyz="0 0 0" rpy="0 0 0" />
                 <mass value="${coxa_mass}" />
                 <xacro:box_inertia mass="${coxa_mass}" x="${coxa_x}"
@@ -157,8 +140,4 @@
         <!-- Gazebo properties -->
         <gazebo reference="leg${leg_number}_coxa">
-            <kp>${coxa_kp}</kp>
-            <kd>${coxa_kd}</kd>
-            <mu1>${coxa_mu1}</mu1>
-            <mu2>${coxa_mu2}</mu2>
             <material>Gazebo/${color}</material>
         </gazebo>
@@ -169,5 +148,5 @@
         <link name="leg${leg_number}_link1">
             <inertial>
-                <origin xyz="0 0 ${pcb_thickness_z / 2}" rpy="0 0 0" />
+                <origin xyz="0 0 0" rpy="0 0 0" />
                 <mass value="${leg_link_1_mass}" />
                 <xacro:box_inertia mass="${leg_link_1_mass}" x="${leg_link_1_x}"
@@ -190,8 +169,4 @@
         <!-- Gazebo properties -->
         <gazebo reference="leg${leg_number}_link1">
-            <kp>${leg_link_1_kp}</kp>
-            <kd>${leg_link_1_kd}</kd>
-            <mu1>${leg_link_1_mu1}</mu1>
-            <mu2>${leg_link_1_mu2}</mu2>
             <material>Gazebo/${color}</material>
         </gazebo>
@@ -202,5 +177,5 @@
         <link name="leg${leg_number}_link2">
             <inertial>
-                <origin xyz="0 0 ${pcb_thickness_z / 2}" rpy="0 0 0" />
+                <origin xyz="0 0 0" rpy="0 0 0" />
                 <mass value="${leg_link_2_mass}" />
                 <xacro:box_inertia mass="${leg_link_2_mass}" x="${leg_link_2_x}"
@@ -223,8 +198,4 @@
         <!-- Gazebo properties -->
         <gazebo reference="leg${leg_number}_link2">
-            <kp>${leg_link_2_kp}</kp>
-            <kd>${leg_link_2_kd}</kd>
-            <mu1>${leg_link_2_mu1}</mu1>
-            <mu2>${leg_link_2_mu2}</mu2>
             <material>Gazebo/${color}</material>
         </gazebo>
@@ -235,5 +206,5 @@
         <link name="leg${leg_number}_link3">
             <inertial>
-                <origin xyz="0 0 ${pcb_thickness_z / 2}" rpy="0 0 0" />
+                <origin xyz="0 0 0" rpy="0 0 0" />
                 <mass value="${leg_link_3_mass}" />
                 <xacro:box_inertia mass="${leg_link_3_mass}" x="${leg_link_3_x}"
@@ -256,8 +227,4 @@
         <!-- Gazebo properties -->
         <gazebo reference="leg${leg_number}_link3">
-            <kp>${leg_link_3_kp}</kp>
-            <kd>${leg_link_3_kd}</kd>
-            <mu1>${leg_link_3_mu1}</mu1>
-            <mu2>${leg_link_3_mu2}</mu2>
             <material>Gazebo/${color}</material>
         </gazebo>
@@ -268,4 +235,10 @@
         <!-- Joint Link Geometry -->
         <link name="leg${leg_number}_joint_link${link_number}">
+            <inertial>
+                <origin xyz="0 0 0" rpy="0 0 0" />
+                <mass value="${joint_link_mass}" />
+                <xacro:cylinder_inerta mass="${joint_link_mass}"
+                    r="${joint_link_r}" l="${joint_link_l}" />
+            </inertial>
             <collision>
                 <origin xyz="0 0 0" rpy="0 0 0" />
@@ -316,5 +289,4 @@
             <child link="leg${leg_number}_joint_link1" />
             <origin xyz="0 ${(coxa_y / 2) + (joint_link_r)} 0" rpy="0 0 0" />
-            <dynamics damping="${joint_damping}" friction="${joint_friction}" />
             <limit lower="${joint_lower_limit}"
                    upper="${joint_upper_limit}"
@@ -341,5 +313,4 @@
             <origin xyz="${-((leg_link_1_x / 2) + (joint_link_r))}
                 ${(leg_link_1_y / 2) - (joint_link_l / 2)} 0" rpy="0 0 0" />
-            <dynamics damping="${joint_damping}" friction="${joint_friction}" />
             <limit lower="${joint_lower_limit}"
                    upper="${joint_upper_limit}"
@@ -366,5 +337,4 @@
             <origin xyz="${-(leg_link_2_x / 2) + (joint_link_l / 2)}
                 ${(leg_link_2_y / 2) + (joint_link_r)} 0" rpy="0 0 0" />
-            <dynamics damping="${joint_damping}" friction="${joint_friction}" />
             <limit lower="${joint_lower_limit}"
                    upper="${joint_upper_limit}"
