Commit message: tuned pid values to minimize vibrations due to commanded joint position.

File: robot/millihex_description.xacro (robot description, xacro)
@@ -13,5 +13,5 @@
     <!-- PCB Properties -->
     <xacro:property name="pcb_density" value="1850" />       <!-- FR4 density (kg/m^3) -->
-    <xacro:property name="pcb_thickness_z" value="0.003" />  <!-- PCB thickness (m) -->
+    <xacro:property name="pcb_thickness_z" value="0.002" />  <!-- PCB thickness (m) -->
     <!-- Thorax Properties -->
     <xacro:property name="thorax_x" value="0.25" />     <!-- x length (m) -->
@@ -40,6 +40,6 @@
         value="${pcb_density * (leg_link_3_x * leg_link_3_y * pcb_thickness_z)}" />  <!-- (kg) -->
     <!-- Joint Link Properties -->
-    <xacro:property name="joint_link_r" value="0.0015" />  <!-- radius (m) -->
-    <xacro:property name="joint_link_l" value="0.01" />    <!-- length (m) -->
+    <xacro:property name="joint_link_r" value="${pcb_thickness_z / 2}" />  <!-- radius (m) -->
+    <xacro:property name="joint_link_l" value="${coxa_x}" />               <!-- length (m) -->
     <xacro:property name="joint_link_mass"
         value="${pcb_density * (pi * (joint_link_r * joint_link_r) * joint_link_l)}" />  <!-- (kg) -->

Commit message: adjusted joint effort and velocity limits.

File: robot/millihex_description.xacro (robot description, xacro)
@@ -48,5 +48,5 @@
     <xacro:property name="joint_lower_limit" value="${-pi / 2}" />  <!-- (rad) -->
     <xacro:property name="joint_effort_limit" value="0.1" />        <!-- (N*m) -->
-    <xacro:property name="joint_velocity_limit" value="${pi / 4}" />      <!-- (rad/s) -->
+    <xacro:property name="joint_velocity_limit" value="0.1" />      <!-- (rad/s) -->
     <!-- Thorax Leg Joint Attachment Positions -->
     <xacro:property name="leg_spacing" value="${(2 * coxa_x) + leg_link_2_x}" />

Commit message: adjusting friction and pid values for tripod gait walking demo.

File: robot/millihex_description.xacro (robot description, xacro)
@@ -37,4 +37,6 @@
     <xacro:property name="leg_link_3_x" value="0.01" />     <!-- x length (m) -->
     <xacro:property name="leg_link_3_y" value="0.05" />     <!-- y length (m) -->
+    <xacro:property name="foot_mu1" value="100.0" />          <!-- friction coefficient 1 -->
+    <xacro:property name="foot_mu2" value="100.0" />          <!-- friction coefficient 2 -->
     <xacro:property name="leg_link_3_mass"
         value="${pcb_density * (leg_link_3_x * leg_link_3_y * pcb_thickness_z)}" />  <!-- (kg) -->
@@ -47,5 +49,5 @@
     <xacro:property name="joint_upper_limit" value="${pi / 2}" />   <!-- (rad) -->
     <xacro:property name="joint_lower_limit" value="${-pi / 2}" />  <!-- (rad) -->
-    <xacro:property name="joint_effort_limit" value="0.1" />        <!-- (N*m) -->
+    <xacro:property name="joint_effort_limit" value="1.0" />        <!-- (N*m) -->
     <xacro:property name="joint_velocity_limit" value="0.1" />      <!-- (rad/s) -->
     <!-- Thorax Leg Joint Attachment Positions -->
@@ -227,4 +229,6 @@
         <!-- Gazebo properties -->
         <gazebo reference="leg${leg_number}_link3">
+            <mu1>${foot_mu1}</mu1>
+            <mu2>${foot_mu2}</mu2>
             <material>Gazebo/${color}</material>
         </gazebo>

Commit message: added back contact stiffness, contact damping, and frictions.

File: robot/millihex_description.xacro (robot description, xacro)
@@ -37,6 +37,4 @@
     <xacro:property name="leg_link_3_x" value="0.01" />     <!-- x length (m) -->
     <xacro:property name="leg_link_3_y" value="0.05" />     <!-- y length (m) -->
-    <xacro:property name="foot_mu1" value="100.0" />          <!-- friction coefficient 1 -->
-    <xacro:property name="foot_mu2" value="100.0" />          <!-- friction coefficient 2 -->
     <xacro:property name="leg_link_3_mass"
         value="${pcb_density * (leg_link_3_x * leg_link_3_y * pcb_thickness_z)}" />  <!-- (kg) -->
@@ -46,9 +44,14 @@
     <xacro:property name="joint_link_mass"
         value="${pcb_density * (pi * (joint_link_r * joint_link_r) * joint_link_l)}" />  <!-- (kg) -->
-    <!-- Revolute Joint Properties -->
+    <!-- Link Friction and -->
+    <xacro:property name="link_kp" value="1000000.0" />  <!-- Contact stiffness -->
+    <xacro:property name="link_kd" value="1.0" />        <!-- Contact damping -->
+    <xacro:property name="link_mu1" value="100.0" />     <!-- Friction coefficient 1 -->
+    <xacro:property name="link_mu2" value="100.0" />     <!-- Friction coefficient 2 -->
+    <!-- Revolute Joint Limits -->
     <xacro:property name="joint_upper_limit" value="${pi / 2}" />   <!-- (rad) -->
     <xacro:property name="joint_lower_limit" value="${-pi / 2}" />  <!-- (rad) -->
-    <xacro:property name="joint_effort_limit" value="1.0" />        <!-- (N*m) -->
-    <xacro:property name="joint_velocity_limit" value="0.1" />      <!-- (rad/s) -->
+    <xacro:property name="joint_effort_limit" value="0.01" />        <!-- (N*m) -->
+    <xacro:property name="joint_velocity_limit" value="0.01" />      <!-- (rad/s) -->
     <!-- Thorax Leg Joint Attachment Positions -->
     <xacro:property name="leg_spacing" value="${(2 * coxa_x) + leg_link_2_x}" />
@@ -108,4 +111,8 @@
         <!-- Gazebo properties -->
         <gazebo reference="thorax">
+            <kp>${link_kp}</kp>
+            <kd>${link_kd}</kd>
+            <mu1>${link_mu1}</mu1>
+            <mu2>${link_mu2}</mu2>
             <material>Gazebo/${color}</material>
         </gazebo>
@@ -142,4 +149,8 @@
         <!-- Gazebo properties -->
         <gazebo reference="leg${leg_number}_coxa">
+            <kp>${link_kp}</kp>
+            <kd>${link_kd}</kd>
+            <mu1>${link_mu1}</mu1>
+            <mu2>${link_mu2}</mu2>
             <material>Gazebo/${color}</material>
         </gazebo>
@@ -171,4 +182,8 @@
         <!-- Gazebo properties -->
         <gazebo reference="leg${leg_number}_link1">
+            <kp>${link_kp}</kp>
+            <kd>${link_kd}</kd>
+            <mu1>${link_mu1}</mu1>
+            <mu2>${link_mu2}</mu2>
             <material>Gazebo/${color}</material>
         </gazebo>
@@ -200,4 +215,8 @@
         <!-- Gazebo properties -->
         <gazebo reference="leg${leg_number}_link2">
+            <kp>${link_kp}</kp>
+            <kd>${link_kd}</kd>
+            <mu1>${link_mu1}</mu1>
+            <mu2>${link_mu2}</mu2>
             <material>Gazebo/${color}</material>
         </gazebo>
@@ -229,6 +248,8 @@
         <!-- Gazebo properties -->
         <gazebo reference="leg${leg_number}_link3">
-            <mu1>${foot_mu1}</mu1>
-            <mu2>${foot_mu2}</mu2>
+            <kp>${link_kp}</kp>
+            <kd>${link_kd}</kd>
+            <mu1>${link_mu1}</mu1>
+            <mu2>${link_mu2}</mu2>
             <material>Gazebo/${color}</material>
         </gazebo>
@@ -261,4 +282,8 @@
         <!-- Gazebo properties -->
         <gazebo reference="leg${leg_number}_joint_link${link_number}">
+            <kp>${link_kp}</kp>
+            <kd>${link_kd}</kd>
+            <mu1>${link_mu1}</mu1>
+            <mu2>${link_mu2}</mu2>
             <material>Gazebo/${color}</material>
         </gazebo>

Commit message: fixed inertia tensor for cylinder macro equation.

File: robot/millihex_description.xacro (robot description, xacro)
@@ -71,5 +71,5 @@
         <color rgba="0.0 0.0 0.0 0.0" />
     </material>
-    <!-- Calculate Moment of Inertia of a Box -->
+    <!-- Calculate Inertia Tensor of a Box -->
     <xacro:macro name="box_inertia" params="mass x y z">
         <inertia ixx="${(1 / 12) * mass * ((y * y) + (z * z))}" ixy = "0" ixz = "0"
@@ -77,9 +77,9 @@
                  izz="${(1 / 12) * mass * ((x * x) + (y * y))}" />
     </xacro:macro>
-    <!-- Calculate Moment of Inertia of a Cylinder -->
+    <!-- Calculate Inertia Tensor of a Cylinder -->
     <xacro:macro name="cylinder_inerta" params="mass r l">
-        <inertia ixx="${(1 / 12) * mass * (l * l)}" ixy = "0" ixz = "0"
-                 iyy="${(1 / 12) * mass * (l * l)}" iyz = "0"
-                 izz="${(1 / 2) * mass * (r * r)}" />
+        <inertia ixx="${(1 / 12) * mass * (3 * (r * r) + (l * l))}" ixy = "0" ixz = "0"
+                 iyy="${(1 / 12) * mass * (3 * (r * r) + (l * l))}" iyz = "0"
+                 izz="${(1 / 12) * mass * (r * r)}" />
     </xacro:macro>
     <!-- Thorax Definition -->
