Commit message: tuned proportional gain and damping parameters for a material density of 2000.

File: robot/millihex_description.xacro (robot description, xacro)
@@ -12,29 +12,29 @@
     </xacro:macro>
     <!-- PCB Properties -->
-    <xacro:property name="pcb_density" value="1850" />       <!-- FR4 density (kg/m^3) -->
+    <xacro:property name="pcb_density" value="2000" />       <!-- FR4 density (kg/m^3) -->
     <xacro:property name="pcb_thickness_z" value="0.002" />  <!-- PCB thickness (m) -->
     <!-- Thorax Properties -->
-    <xacro:property name="thorax_x" value="0.25" />     <!-- x length (m) -->
+    <xacro:property name="thorax_x" value="0.17" />     <!-- x length (m) -->
     <xacro:property name="thorax_y" value="0.02" />     <!-- y length (m) -->
     <xacro:property name="thorax_mass"
         value="${pcb_density * (thorax_x * thorax_y * pcb_thickness_z)}" />  <!-- (kg) -->
     <!-- Coxa Properties -->
-    <xacro:property name="coxa_x" value="0.01" />     <!-- x length (m) -->
-    <xacro:property name="coxa_y" value="0.01" />     <!-- y length (m) -->
+    <xacro:property name="coxa_x" value="0.015" />     <!-- x length (m) -->
+    <xacro:property name="coxa_y" value="0.015" />     <!-- y length (m) -->
     <xacro:property name="coxa_mass"
         value="${pcb_density * (coxa_x * coxa_y * pcb_thickness_z)}" />  <!-- (kg) -->
     <!-- Femur (Leg Link 1) Properties -->
-    <xacro:property name="leg_link1_x" value="0.01" />     <!-- x length (m) -->
-    <xacro:property name="leg_link1_y" value="0.05" />     <!-- y length (m) -->
+    <xacro:property name="leg_link1_x" value="0.015" />     <!-- x length (m) -->
+    <xacro:property name="leg_link1_y" value="0.03" />     <!-- y length (m) -->
     <xacro:property name="leg_link1_mass"
         value="${pcb_density * (leg_link1_x * leg_link1_y * pcb_thickness_z)}" />  <!-- (kg) -->
     <!-- Tibia (Leg Link 2) Properties -->
-    <xacro:property name="leg_link2_x" value="0.05" />     <!-- x length (m) -->
-    <xacro:property name="leg_link2_y" value="0.01" />     <!-- y length (m) -->
+    <xacro:property name="leg_link2_x" value="0.02" />     <!-- x length (m) -->
+    <xacro:property name="leg_link2_y" value="0.015" />     <!-- y length (m) -->
     <xacro:property name="leg_link2_mass"
         value="${pcb_density * (leg_link2_x * leg_link2_y * pcb_thickness_z)}" />  <!-- (kg) -->
     <!-- Tarsus (Leg Link 3) Properties -->
-    <xacro:property name="leg_link3_x" value="0.01" />     <!-- x length (m) -->
-    <xacro:property name="leg_link3_y" value="0.05" />     <!-- y length (m) -->
+    <xacro:property name="leg_link3_x" value="0.015" />     <!-- x length (m) -->
+    <xacro:property name="leg_link3_y" value="0.03" />     <!-- y length (m) -->
     <xacro:property name="leg_link3_mass"
         value="${pcb_density * (leg_link3_x * leg_link3_y * pcb_thickness_z)}" />  <!-- (kg) -->
@@ -45,13 +45,15 @@
         value="${pcb_density * (pi * (joint_link_r * joint_link_r) * joint_link_l)}" />  <!-- (kg) -->
     <!-- Link Friction and -->
-    <xacro:property name="link_kp" value="1000000.0" />  <!-- Contact stiffness -->
-    <xacro:property name="link_kd" value="100.0" />        <!-- Contact damping -->
-    <xacro:property name="link_mu1" value="100.0" />     <!-- Friction coefficient 1 -->
-    <xacro:property name="link_mu2" value="100.0" />     <!-- Friction coefficient 2 -->
-    <!-- Revolute Joint Limits -->
+    <xacro:property name="link_kp" value="1000.0" />  <!-- Contact stiffness -->
+    <xacro:property name="link_kd" value="1.0" />        <!-- Contact damping -->
+    <xacro:property name="link_mu1" value="10.0" />     <!-- Friction coefficient 1 -->
+    <xacro:property name="link_mu2" value="10.0" />     <!-- Friction coefficient 2 -->
+    <!-- Revolute Joint Properties -->
     <xacro:property name="joint_upper_limit" value="${pi / 2}" />   <!-- (rad) -->
     <xacro:property name="joint_lower_limit" value="${-pi / 2}" />  <!-- (rad) -->
     <xacro:property name="joint_effort_limit" value="1.0" />        <!-- (N*m) -->
     <xacro:property name="joint_velocity_limit" value="1.0" />      <!-- (rad/s) -->
+    <xacro:property name="joint_damping" value="4.6e-6" />        <!-- (N*m*s/rad) -->
+    <xacro:property name="joint_friction" value="0.0" />            <!-- (N*m) -->
     <!-- Thorax Leg Joint Attachment Positions -->
     <xacro:property name="leg_spacing" value="${(2 * coxa_x) + leg_link2_x}" />
@@ -165,5 +167,5 @@
             </inertial>
             <collision>
-                <origin xyz="0 ${leg_link1_y / 2} 0" rpy="0 0 0" />
+                <origin xyz="0 ${(leg_link1_y / 2) + joint_link_r} 0" rpy="0 0 0" />
                 <geometry>
                     <box size="${leg_link1_x} ${leg_link1_y} ${pcb_thickness_z}" />
@@ -171,5 +173,5 @@
             </collision>
             <visual>
-                <origin xyz="0 ${leg_link1_y / 2} 0" rpy="0 0 0" />
+                <origin xyz="0 ${(leg_link1_y / 2) + joint_link_r} 0" rpy="0 0 0" />
                 <geometry>
                     <box size="${leg_link1_x} ${leg_link1_y} ${pcb_thickness_z}" />
@@ -198,5 +200,5 @@
             </inertial>
             <collision>
-                <origin xyz="${-leg_link2_x / 2} 0 0" rpy="0 0 0" />
+                <origin xyz="${-((leg_link2_x / 2) + joint_link_r)} 0 0" rpy="0 0 0" />
                 <geometry>
                     <box size="${leg_link2_x} ${leg_link2_y} ${pcb_thickness_z}" />
@@ -204,5 +206,5 @@
             </collision>
             <visual>
-                <origin xyz="${-leg_link2_x / 2} 0 0" rpy="0 0 0" />
+                <origin xyz="${-((leg_link2_x / 2) + joint_link_r)} 0 0" rpy="0 0 0" />
                 <geometry>
                     <box size="${leg_link2_x} ${leg_link2_y} ${pcb_thickness_z}" />
@@ -231,5 +233,5 @@
             </inertial>
             <collision>
-                <origin xyz="0 ${leg_link3_y / 2} 0" rpy="0 0 0" />
+                <origin xyz="0 ${(leg_link3_y / 2) + joint_link_r} 0" rpy="0 0 0" />
                 <geometry>
                     <box size="${leg_link3_x} ${leg_link3_y} ${pcb_thickness_z}" />
@@ -237,5 +239,5 @@
             </collision>
             <visual>
-                <origin xyz="0 ${leg_link3_y / 2} 0" rpy="0 0 0" />
+                <origin xyz="0 ${(leg_link3_y / 2) + joint_link_r} 0" rpy="0 0 0" />
                 <geometry>
                     <box size="${leg_link3_x} ${leg_link3_y} ${pcb_thickness_z}" />
@@ -264,10 +266,4 @@
                     r="${joint_link_r}" l="${joint_link_l}" />
             </inertial>
-            <collision>
-                <origin xyz="0 0 0" rpy="0 0 0" />
-                <geometry>
-                    <cylinder radius="${joint_link_r}" length="${joint_link_l}" />
-                </geometry>
-            </collision>
             <visual>
                 <origin xyz="0 0 0" rpy="0 ${pi / 2} ${yaw}" />
@@ -316,4 +312,5 @@
             <child link="leg${leg_number}_joint_link1" />
             <origin xyz="0 ${coxa_y + joint_link_r} 0" rpy="0 0 0" />
+            <dynamics damping="${joint_damping}" friction="${joint_friction}"/>
             <limit lower="${joint_lower_limit}"
                    upper="${joint_upper_limit}"
@@ -329,5 +326,5 @@
             <parent link="leg${leg_number}_joint_link1" />
             <child link="leg${leg_number}_link1" />
-            <origin xyz="0 ${joint_link_r} 0" rpy="0 0 0" />
+            <origin xyz="0 0 0" rpy="0 0 0" />
         </joint>
         <!-- Joint Link 2 -->
@@ -339,5 +336,7 @@
             <child link="leg${leg_number}_joint_link2" />
             <origin xyz="${-((leg_link1_x / 2) + joint_link_r)}
-                ${(leg_link1_y) - (joint_link_l / 2)} 0" rpy="0 0 0" />
+                ${(leg_link1_y) - (joint_link_l / 2) + joint_link_r} 0"
+                rpy="0 0 0" />
+            <dynamics damping="${joint_damping}" friction="${joint_friction}"/>
             <limit lower="${joint_lower_limit}"
                    upper="${joint_upper_limit}"
@@ -353,5 +352,5 @@
             <parent link="leg${leg_number}_joint_link2" />
             <child link="leg${leg_number}_link2" />
-            <origin xyz="${-joint_link_r} 0 0" rpy="0 0 0" />
+            <origin xyz="0 0 0" rpy="0 0 0" />
         </joint>
         <!-- Joint Link 3 -->
@@ -362,6 +361,7 @@
             <parent link="leg${leg_number}_link2" />
             <child link="leg${leg_number}_joint_link3" />
-            <origin xyz="${-(leg_link2_x) + (joint_link_l / 2)}
+            <origin xyz="${-(leg_link2_x) + (joint_link_l / 2) - joint_link_r}
                 ${(leg_link2_y / 2) + joint_link_r} 0" rpy="0 0 0" />
+            <dynamics damping="${joint_damping}" friction="${joint_friction}"/>
             <limit lower="${joint_lower_limit}"
                    upper="${joint_upper_limit}"
@@ -377,5 +377,5 @@
             <parent link="leg${leg_number}_joint_link3" />
             <child link="leg${leg_number}_link3" />
-            <origin xyz="0 ${joint_link_r} 0" rpy="0 0 0" />
+            <origin xyz="0 0 0" rpy="0 0 0" />
         </joint>
     </xacro:macro>

Commit message: Added back collision to joint link. Playing with gait demo.

File: robot/millihex_description.xacro (robot description, xacro)
@@ -266,4 +266,10 @@
                     r="${joint_link_r}" l="${joint_link_l}" />
             </inertial>
+            <collision>
+                <origin xyz="0 0 0" rpy="0 ${pi / 2} ${yaw}" />
+                <geometry>
+                    <cylinder radius="${joint_link_r}" length="${joint_link_l}" />
+                </geometry>
+            </collision>
             <visual>
                 <origin xyz="0 0 0" rpy="0 ${pi / 2} ${yaw}" />

Commit message: More PID tweaks with new link geometry and joint_link collision. Added 100 Hz joint movement sequence in demo.

File: robot/millihex_description.xacro (robot description, xacro)
@@ -45,8 +45,8 @@
         value="${pcb_density * (pi * (joint_link_r * joint_link_r) * joint_link_l)}" />  <!-- (kg) -->
     <!-- Link Friction and -->
-    <xacro:property name="link_kp" value="1000.0" />  <!-- Contact stiffness -->
+    <xacro:property name="link_kp" value="100000.0" />  <!-- Contact stiffness -->
     <xacro:property name="link_kd" value="1.0" />        <!-- Contact damping -->
-    <xacro:property name="link_mu1" value="10.0" />     <!-- Friction coefficient 1 -->
-    <xacro:property name="link_mu2" value="10.0" />     <!-- Friction coefficient 2 -->
+    <xacro:property name="link_mu1" value="100.0" />     <!-- Friction coefficient 1 -->
+    <xacro:property name="link_mu2" value="100.0" />     <!-- Friction coefficient 2 -->
     <!-- Revolute Joint Properties -->
     <xacro:property name="joint_upper_limit" value="${pi / 2}" />   <!-- (rad) -->
@@ -54,5 +54,5 @@
     <xacro:property name="joint_effort_limit" value="1.0" />        <!-- (N*m) -->
     <xacro:property name="joint_velocity_limit" value="1.0" />      <!-- (rad/s) -->
-    <xacro:property name="joint_damping" value="4.6e-6" />        <!-- (N*m*s/rad) -->
+    <xacro:property name="joint_damping" value="0.0" />        <!-- (N*m*s/rad) -->
     <xacro:property name="joint_friction" value="0.0" />            <!-- (N*m) -->
     <!-- Thorax Leg Joint Attachment Positions -->

Commit message: Working on vectorized set_joint_positions function.

File: robot/millihex_description.xacro (robot description, xacro)
@@ -323,5 +323,5 @@
                    effort="${joint_effort_limit}"
                    velocity="${joint_velocity_limit}" />
-            <axis xyz="-1 0 0" />
+            <axis xyz="1 0 0" />
         </joint>
         <xacro:leg_transmission leg_number="${leg_number}" joint_number="1" />
@@ -349,5 +349,5 @@
                    effort="${joint_effort_limit}"
                    velocity="${joint_velocity_limit}" />
-            <axis xyz="0 -1 0" />
+            <axis xyz="0 1 0" />
         </joint>
         <xacro:leg_transmission leg_number="${leg_number}" joint_number="2" />
@@ -374,5 +374,5 @@
                    effort="${joint_effort_limit}"
                    velocity="${joint_velocity_limit}" />
-            <axis xyz="-1 0 0" />
+            <axis xyz="1 0 0" />
         </joint>
         <xacro:leg_transmission leg_number="${leg_number}" joint_number="3" />

Commit message: Added foot joint to serve as end effector.

File: robot/millihex_description.xacro (robot description, xacro)
@@ -385,4 +385,13 @@
             <origin xyz="0 0 0" rpy="0 0 0" />
         </joint>
+        <!-- Joint Link 4 (Foot) -->
+        <xacro:millihex_joint_link leg_number="${leg_number}" link_number="4"
+            yaw="0.0" color="White" />
+        <!-- Fixed Joint 4 (Foot Joint) -->
+        <joint name="leg${leg_number}_fixed_joint4" type="fixed">
+            <parent link="leg${leg_number}_link3" />
+            <child link="leg${leg_number}_joint_link4" />
+            <origin xyz="0 ${leg_link3_y + (2 * joint_link_r)} 0" rpy="0 0 0" />
+        </joint>
     </xacro:macro>
     <!-- Assemble Body -->
