Commit message: Obstacle xacro and launch file now parameterized. Need to add friction to obstacle.

File: models/obstacle_description.xacro (robot description, xacro)
@@ -3,28 +3,47 @@
 <!-- rosrun xacro xacro obstacle_description.xacro > obstacle_description.urdf -->
 <robot name="obstacle" xmlns:xacro="http://www.ros.org/wiki/xacro">
-    <xacro:arg name="x_arg" default="10"/>
-    <xacro:property name="x_property" value="$(arg x_arg)" />
+    <!-- Obstacle Parameters -->
+    <xacro:arg name="l" default="1"/>
+    <xacro:arg name="w" default="1"/>
+    <xacro:arg name="h" default="1"/>
+    <xacro:arg name="d" default="1"/>
+    <!-- Calculate Inertia Tensor of a Box -->
+    <xacro:macro name="box_inertia" params="mass x y z">
+        <inertia ixx="${(1 / 12) * mass * ((y * y) + (z * z))}" ixy = "0" ixz = "0"
+                 iyy="${(1 / 12) * mass * ((x * x) + (z * z))}" iyz = "0"
+                 izz="${(1 / 12) * mass * ((x * x) + (y * y))}" />
+    </xacro:macro>
     <link name="box">
         <inertial>
-            <origin xyz="2 0 0" />
+            <origin xyz="0 0 0" rpy="0 0 0" />
             <mass value="1.0" />
-            <inertia  ixx="1.0" ixy="0.0"  ixz="0.0"  iyy="100.0"  iyz="0.0"  izz="1.0" />
+            <inertia  ixx="1.0" ixy="0.0"  ixz="0.0"  iyy="1.0"  iyz="0.0"  izz="1.0" />
         </inertial>
         <visual>
-            <origin xyz="2 0 1"/>
+            <origin xyz="$(arg d) 0 0" rpy="0 0 0" />
             <geometry>
-                <box size="1 1 2" />
+                <box size="$(arg l) $(arg w) $(arg h)" />
             </geometry>
         </visual>
         <collision>
-            <origin xyz="2 0 1"/>
+            <origin xyz="$(arg d) 0 0" rpy="0 0 0" />
             <geometry>
-                <box size="1 1 2" />
+                <box size="$(arg l) $(arg w) $(arg h)" />
             </geometry>
         </collision>
     </link>
+    <!-- Fix the Obstacle to world -->
+    <link name="world"/>
+    <joint name="fixed" type="fixed">
+        <parent link="world"/>
+        <child link="box"/>
+    </joint>
     <!-- Gazebo properties -->
     <gazebo reference="box">
         <material>Gazebo/Blue</material>
     </gazebo>
+    <!-- Make Obstacle stationary -->
+    <gazebo>
+        <static>true</static>
+    </gazebo>
 </robot>

Commit message: Added walls to obstacle URDF.

File: models/obstacle_description.xacro (robot description, xacro)
@@ -4,13 +4,13 @@
 <robot name="obstacle" xmlns:xacro="http://www.ros.org/wiki/xacro">
     <!-- Obstacle Parameters -->
-    <xacro:arg name="l" default="1"/>
-    <xacro:arg name="w" default="1"/>
-    <xacro:arg name="h" default="1"/>
-    <xacro:arg name="d" default="1"/>
+    <xacro:arg name="l" default="0.2"/>
+    <xacro:arg name="w" default="0.5"/>
+    <xacro:arg name="h" default="0.02"/>
+    <xacro:arg name="d" default="0.3"/>
     <!-- Wall Parameters -->
     <xacro:property name="wall_l" value="0.01" />
-    <xacro:property name="wall_w" value="0.5" />
     <xacro:property name="wall_h" value="0.2" />
-    <xacro:property name="wall_d" value="${wall_w / 2}" />
+    <xacro:property name="back_wall_w" value="0.5" />
+    <xacro:property name="side_wall_w" value="0.65" />
     <!-- Define world link -->
     <link name="world"/>
@@ -56,13 +56,13 @@
         </inertial>
         <visual>
-            <origin xyz="${-wall_d} 0 0" rpy="0 0 0" />
+            <origin xyz="${-back_wall_w/2 + 0.005} 0 0" rpy="0 0 0" />
             <geometry>
-                <box size="${wall_l} ${wall_w} ${wall_h}" />
+                <box size="${wall_l} ${back_wall_w} ${wall_h}" />
             </geometry>
         </visual>
         <collision>
-            <origin xyz="${-wall_d} 0" rpy="0 0 0" />
+            <origin xyz="${-back_wall_w/2 + 0.005} 0 0" rpy="0 0 0" />
             <geometry>
-                <box size="${wall_l} ${wall_w} ${wall_h}" />
+                <box size="${wall_l} ${back_wall_w} ${wall_h}" />
             </geometry>
         </collision>
@@ -85,13 +85,13 @@
         </inertial>
         <visual>
-            <origin xyz="0 ${wall_d} 0" rpy="0 0 ${pi/2}" />
+            <origin xyz="0.075 ${back_wall_w/2} 0" rpy="0 0 ${pi/2}" />
             <geometry>
-                <box size="${wall_l} ${wall_w} ${wall_h}" />
+                <box size="${wall_l} ${side_wall_w} ${wall_h}" />
             </geometry>
         </visual>
         <collision>
-            <origin xyz="0 ${wall_d} 0" rpy="0 0 ${pi/2}" />
+            <origin xyz="0.075 ${back_wall_w/2} 0" rpy="0 0 ${pi/2}" />
             <geometry>
-                <box size="${wall_l} ${wall_w} ${wall_h}" />
+                <box size="${wall_l} ${side_wall_w} ${wall_h}" />
             </geometry>
         </collision>
@@ -114,13 +114,13 @@
         </inertial>
         <visual>
-            <origin xyz="0 ${-wall_d} 0" rpy="0 0 ${pi/2}" />
+            <origin xyz="0.075 ${-back_wall_w/2} 0" rpy="0 0 ${pi/2}" />
             <geometry>
-                <box size="${wall_l} ${wall_w} ${wall_h}" />
+                <box size="${wall_l} ${side_wall_w} ${wall_h}" />
             </geometry>
         </visual>
         <collision>
-            <origin xyz="0 ${-wall_d} 0" rpy="0 0 ${pi/2}" />
+            <origin xyz="0.075 ${-back_wall_w/2} 0" rpy="0 0 ${pi/2}" />
             <geometry>
-                <box size="${wall_l} ${wall_w} ${wall_h}" />
+                <box size="${wall_l} ${side_wall_w} ${wall_h}" />
             </geometry>
         </collision>

Commit message: Testing faster gait and friction parameters. May need to use SDF...

File: models/obstacle_description.xacro (robot description, xacro)
@@ -8,4 +8,9 @@
     <xacro:arg name="h" default="0.02"/>
     <xacro:arg name="d" default="0.3"/>
+    <!-- Obstacle Friction -->
+    <xacro:property name="kp" value="100000.0" />  <!-- Contact stiffness -->
+    <xacro:property name="kd" value="1.0" />        <!-- Contact damping -->
+    <xacro:property name="mu1" value="1000.0" />     <!-- Friction coefficient 1 -->
+    <xacro:property name="mu2" value="1000.0" />     <!-- Friction coefficient 2 -->
     <!-- Wall Parameters -->
     <xacro:property name="wall_l" value="0.01" />
@@ -46,4 +51,8 @@
     <!-- Gazebo properties -->
     <gazebo reference="obstacle">
+        <kp>${kp}</kp>
+        <kd>${kd}</kd>
+        <mu1>${mu1}</mu1>
+        <mu2>${mu2}</mu2>
         <material>Gazebo/White</material>
     </gazebo>

Commit message: Added launch file to separate spawning of room and obstacle. start_gazebo launch file now spawns the room. The object spawns separately to enable automated testing.

File: models/obstacle_description.xacro (robot description, xacro)
@@ -13,9 +13,4 @@
     <xacro:property name="mu1" value="1000.0" />     <!-- Friction coefficient 1 -->
     <xacro:property name="mu2" value="1000.0" />     <!-- Friction coefficient 2 -->
-    <!-- Wall Parameters -->
-    <xacro:property name="wall_l" value="0.01" />
-    <xacro:property name="wall_h" value="0.2" />
-    <xacro:property name="back_wall_w" value="0.5" />
-    <xacro:property name="side_wall_w" value="0.65" />
     <!-- Define world link -->
     <link name="world"/>
@@ -57,90 +52,3 @@
         <material>Gazebo/White</material>
     </gazebo>
-    <!-- Back Wall -->
-    <link name="back_wall">
-        <inertial>
-            <origin xyz="0 0 0" rpy="0 0 0" />
-            <mass value="1.0" />
-            <inertia  ixx="1.0" ixy="0.0"  ixz="0.0"  iyy="1.0"  iyz="0.0"  izz="1.0" />
-        </inertial>
-        <visual>
-            <origin xyz="${-back_wall_w/2 + 0.005} 0 0" rpy="0 0 0" />
-            <geometry>
-                <box size="${wall_l} ${back_wall_w} ${wall_h}" />
-            </geometry>
-        </visual>
-        <collision>
-            <origin xyz="${-back_wall_w/2 + 0.005} 0 0" rpy="0 0 0" />
-            <geometry>
-                <box size="${wall_l} ${back_wall_w} ${wall_h}" />
-            </geometry>
-        </collision>
-    </link>
-    <!-- Fix Back Wall to world -->
-    <joint name="back_wall_fixed_joint" type="fixed">
-        <parent link="world"/>
-        <child link="back_wall"/>
-    </joint>
-    <!-- Gazebo properties -->
-    <gazebo reference="back_wall">
-        <material>Gazebo/White</material>
-    </gazebo>
-    <!-- Left Wall -->
-    <link name="left_wall">
-        <inertial>
-            <origin xyz="0 0 0" rpy="0 0 0" />
-            <mass value="1.0" />
-            <inertia  ixx="1.0" ixy="0.0"  ixz="0.0"  iyy="1.0"  iyz="0.0"  izz="1.0" />
-        </inertial>
-        <visual>
-            <origin xyz="0.075 ${back_wall_w/2} 0" rpy="0 0 ${pi/2}" />
-            <geometry>
-                <box size="${wall_l} ${side_wall_w} ${wall_h}" />
-            </geometry>
-        </visual>
-        <collision>
-            <origin xyz="0.075 ${back_wall_w/2} 0" rpy="0 0 ${pi/2}" />
-            <geometry>
-                <box size="${wall_l} ${side_wall_w} ${wall_h}" />
-            </geometry>
-        </collision>
-    </link>
-    <!-- Fix Left Wall to world -->
-    <joint name="left_wall_fixed_joint" type="fixed">
-        <parent link="world"/>
-        <child link="left_wall"/>
-    </joint>
-    <!-- Gazebo properties -->
-    <gazebo reference="left_wall">
-        <material>Gazebo/White</material>
-    </gazebo>
-    <!-- Right Wall -->
-    <link name="right_wall">
-        <inertial>
-            <origin xyz="0 0 0" rpy="0 0 0" />
-            <mass value="1.0" />
-            <inertia  ixx="1.0" ixy="0.0"  ixz="0.0"  iyy="1.0"  iyz="0.0"  izz="1.0" />
-        </inertial>
-        <visual>
-            <origin xyz="0.075 ${-back_wall_w/2} 0" rpy="0 0 ${pi/2}" />
-            <geometry>
-                <box size="${wall_l} ${side_wall_w} ${wall_h}" />
-            </geometry>
-        </visual>
-        <collision>
-            <origin xyz="0.075 ${-back_wall_w/2} 0" rpy="0 0 ${pi/2}" />
-            <geometry>
-                <box size="${wall_l} ${side_wall_w} ${wall_h}" />
-            </geometry>
-        </collision>
-    </link>
-    <!-- Fix Right Wall to world -->
-    <joint name="right_wall_fixed_joint" type="fixed">
-        <parent link="world"/>
-        <child link="right_wall"/>
-    </joint>
-    <!-- Gazebo properties -->
-    <gazebo reference="right_wall">
-        <material>Gazebo/White</material>
-    </gazebo>
 </robot>

Commit message: Added quadruped and pentapod gait patterns.

File: models/obstacle_description.xacro (robot description, xacro)
@@ -11,6 +11,6 @@
     <xacro:property name="kp" value="100000.0" />  <!-- Contact stiffness -->
     <xacro:property name="kd" value="1.0" />        <!-- Contact damping -->
-    <xacro:property name="mu1" value="1000.0" />     <!-- Friction coefficient 1 -->
-    <xacro:property name="mu2" value="1000.0" />     <!-- Friction coefficient 2 -->
+    <xacro:property name="mu1" value="100.0" />     <!-- Friction coefficient 1 -->
+    <xacro:property name="mu2" value="100.0" />     <!-- Friction coefficient 2 -->
     <!-- Define world link -->
     <link name="world"/>

Commit message: Increased friction on floor and obstacle.

File: models/obstacle_description.xacro (robot description, xacro)
@@ -10,7 +10,7 @@
     <!-- Obstacle Friction -->
     <xacro:property name="kp" value="100000.0" />  <!-- Contact stiffness -->
-    <xacro:property name="kd" value="1.0" />        <!-- Contact damping -->
-    <xacro:property name="mu1" value="100.0" />     <!-- Friction coefficient 1 -->
-    <xacro:property name="mu2" value="100.0" />     <!-- Friction coefficient 2 -->
+    <xacro:property name="kd" value="100000.0" />      <!-- Contact damping -->
+    <xacro:property name="mu1" value="100000.0" /> <!-- Friction coefficient 1 -->
+    <xacro:property name="mu2" value="100000.0" /> <!-- Friction coefficient 2 -->
     <!-- Define world link -->
     <link name="world"/>

File: models/room_description.xacro (robot description, xacro)
@@ -8,4 +8,10 @@
     <xacro:property name="back_wall_w" value="0.5" />
     <xacro:property name="side_wall_w" value="0.65" />
+    <xacro:property name="floor_h" value="0.005" />
+    <!-- Floor Friction -->
+    <xacro:property name="kp" value="100000.0" />  <!-- Contact stiffness -->
+    <xacro:property name="kd" value="100000.0" />      <!-- Contact damping -->
+    <xacro:property name="mu1" value="100000.0" /> <!-- Friction coefficient 1 -->
+    <xacro:property name="mu2" value="100000.0" /> <!-- Friction coefficient 2 -->
     <!-- Define world link -->
     <link name="world"/>
@@ -101,3 +107,36 @@
         <material>Gazebo/White</material>
     </gazebo>
+    <!-- Floor -->
+    <link name="floor">
+        <inertial>
+            <origin xyz="0 0 0" rpy="0 0 0" />
+            <mass value="1.0" />
+            <inertia  ixx="1.0" ixy="0.0"  ixz="0.0"  iyy="1.0"  iyz="0.0"  izz="1.0" />
+        </inertial>
+        <visual>
+            <origin xyz="0.075 0 0" rpy="0 0 0" />
+            <geometry>
+                <box size="${side_wall_w} ${back_wall_w} ${floor_h}" />
+            </geometry>
+        </visual>
+        <collision>
+            <origin xyz="0.075 0 0" rpy="0 0 0" />
+            <geometry>
+                <box size="${side_wall_w} ${back_wall_w} ${floor_h}" />
+            </geometry>
+        </collision>
+    </link>
+    <!-- Fix Floor to world -->
+    <joint name="floor_fixed_joint" type="fixed">
+        <parent link="world"/>
+        <child link="floor"/>
+    </joint>
+    <!-- Gazebo properties -->
+    <gazebo reference="floor">
+        <kp>${kp}</kp>
+        <kd>${kd}</kd>
+        <mu1>${mu1}</mu1>
+        <mu2>${mu2}</mu2>
+        <material>Gazebo/Grey</material>
+    </gazebo>
 </robot>
