Commit message: Defined min and max range for all parameters. Added automated parameter sweep code in demo script.

File: models/room_description.xacro (robot description, xacro)
@@ -5,5 +5,5 @@
     <!-- Wall Parameters -->
     <xacro:property name="wall_l" value="0.01" />
-    <xacro:property name="wall_h" value="0.2" />
+    <xacro:property name="wall_h" value="0.15" />
     <xacro:property name="back_wall_w" value="0.5" />
     <xacro:property name="side_wall_w" value="0.65" />

Commit message: Playing around with SQL Python in preparation for storing data into a database table.

File: models/room_description.xacro (robot description, xacro)
@@ -8,5 +8,5 @@
     <xacro:property name="back_wall_w" value="0.5" />
     <xacro:property name="side_wall_w" value="0.65" />
-    <xacro:property name="floor_h" value="0.005" />
+    <xacro:property name="floor_h" value="0.001" />
     <!-- Floor Friction -->
     <xacro:property name="kp" value="100000.0" />  <!-- Contact stiffness -->
